Commit message: Fixed several issues with raisim implementation, dealing with loop closure bug

File: hopper_mpc/res/hopper_rev08/hopper_rev08_closed.urdf (robot description, URDF)
Before this commit: robot hopper_rev08, 8 links, 7 joints
Joints:
- added joint Joint 4: type revolute, parent Link 1, child Link 3, origin xyz=0.27 0 0 rpy=-3.1416 -1.0768 3.1416, axis 0 -1 0, limit lower=-1.57 upper=1.57 effort=50 velocity=2000
- joint Joint 0: limit lower=-3.14 upper=3.14 effort=50 velocity=1000 -> lower=-3.14 upper=3.14 effort=50 velocity=2000
- joint Joint 1: limit lower=-0.7597 upper=1.8295 effort=0 velocity=1000 -> lower=-0.7597 upper=1.8295 effort=50 velocity=2000
- joint Joint 2: limit lower=-3.14 upper=3.14 effort=50 velocity=1000 -> lower=-3.14 upper=3.14 effort=50 velocity=2000
- joint Joint 3: limit lower=-1.8295 upper=0.7597 effort=0 velocity=1000 -> lower=-1.8295 upper=0.7597 effort=50 velocity=2000
