Commit message: Successful test of leg inverse kinematic control tracing circle

File: hopper_mpc/res/hopper_rev08/hopper_rev08.urdf (robot description, URDF)
Before this commit: robot hopper_rev08, 8 links, 7 joints
Links:
- link Link 0: geometry collision mesh filename=Link 0.obj; visual mesh filename=Link 0.obj
- link Link 1: geometry collision mesh filename=Link 1.obj; visual mesh filename=Link 1.obj
- link Link 2: geometry collision mesh filename=Link 2.obj; visual mesh filename=Link 2.obj
- link Link 3: geometry collision mesh filename=Link 3.obj; visual mesh filename=Link 3.obj
- link base_link: geometry collision mesh filename=base_link.obj; visual mesh filename=base_link.obj
- link rw0: geometry collision mesh filename=rw0.obj; visual mesh filename=rw0.obj
- link rw1: geometry collision mesh filename=rw1.obj; visual mesh filename=rw1.obj
- link rwz: geometry collision mesh filename=rwz.obj; visual mesh filename=rwz.obj
Joints:
- added joint Joint 4: type revolute, parent Link 1, child Link 3, origin xyz=0.27 0 0 rpy=-3.1416 -1.0768 3.1416, axis 0 -1 0, limit lower=-1.57 upper=1.57 effort=50 velocity=2000
- joint Joint 0: limit lower=-3.14 upper=3.14 effort=0 velocity=0 -> lower=-3.14 upper=3.14 effort=50 velocity=2000
- joint Joint 1: limit lower=-0.7597 upper=1.8295 effort=0 velocity=0 -> lower=-0.7597 upper=1.8295 effort=50 velocity=2000
- joint Joint 2: limit lower=-3.14 upper=3.14 effort=0 velocity=0 -> lower=-3.14 upper=3.14 effort=50 velocity=2000
- joint Joint 3: limit lower=-1.8295 upper=0.7597 effort=0 velocity=0 -> lower=-1.8295 upper=0.7597 effort=50 velocity=2000
